Commit message: renamed package in urdf file, moved meshes to match path in urdf

File: src/omni/urdf/omni.urdf (robot description, URDF)
Before this commit: robot phantom_omni, 7 links, 6 joints
Links:
- link base: geometry visual mesh filename=package://omni/meshes/base.stl
- link lower_arm: geometry visual mesh filename=package://omni/meshes/lower_arm.stl
- link stylus: geometry visual mesh filename=package://omni/meshes/stylus.stl
- link tip: geometry visual mesh filename=package://omni/meshes/tip.stl
- link torso: geometry visual mesh filename=package://omni/meshes/torso.stl
- link upper_arm: geometry visual mesh filename=package://omni/meshes/upper_arm.stl
- link wrist: geometry visual mesh filename=package://omni/meshes/wrist.stl

Commit message: Updated stl file path names.

File: src/omni/urdf/omni.urdf (robot description, URDF)
Before this commit: robot phantom_omni, 7 links, 6 joints
Links:
- link base: geometry visual mesh filename=/ros2_ws/src/SlicerRos2/models/meshes/base.stl
- link lower_arm: geometry visual mesh filename=/ros2_ws/src/SlicerRos2/models/meshes/lower_arm.stl
- link stylus: geometry visual mesh filename=/ros2_ws/src/SlicerRos2/models/meshes/stylus.stl
- link tip: geometry visual mesh filename=/ros2_ws/src/SlicerRos2/models/meshes/tip.stl
- link torso: geometry visual mesh filename=/ros2_ws/src/SlicerRos2/models/meshes/torso.stl
- link upper_arm: geometry visual mesh filename=/ros2_ws/src/SlicerRos2/models/meshes/upper_arm.stl
- link wrist: geometry visual mesh filename=/ros2_ws/src/SlicerRos2/models/meshes/wrist.stl
