Commit message: Updates: * renamed package to sensable_omni_model * use ROS 2 `joint_state_publisher` node to allow joint_state from different topic names * renamed emulation script to `pretend_omni_joint_state_publisher` * updated README.md Still have to figure out namespace and option to skip `joint_state_publisher` if not needed (e.g. if using `joint_state_publisher_gui`)

File: urdf/omni.urdf (robot description, URDF)
Before this commit: robot phantom_omni, 7 links, 6 joints
Links:
- link base: geometry visual mesh filename=package://sensable_omni_model/meshes/base.stl
- link lower_arm: geometry visual mesh filename=package://sensable_omni_model/meshes/lower_arm.stl
- link stylus: geometry visual mesh filename=package://sensable_omni_model/meshes/stylus.stl
- link tip: geometry visual mesh filename=package://sensable_omni_model/meshes/tip.stl
- link torso: geometry visual mesh filename=package://sensable_omni_model/meshes/torso.stl
- link upper_arm: geometry visual mesh filename=package://sensable_omni_model/meshes/upper_arm.stl
- link wrist: geometry visual mesh filename=package://sensable_omni_model/meshes/wrist.stl

Commit message: Minor fixes for USB Touch

File: urdf/omni.urdf (robot description, URDF)
Before this commit: robot phantom_omni, 7 links, 6 joints
Joints:
- joint pitch: origin xyz=0 0.0525 0 rpy=0.5 0 0 -> xyz=0 0.0525 0 rpy=1.5707 0 0
